File: 2G5_FMC_Test_Board_V1/2G5_FMC_Test_Board_V1.kicad_sch (KiCad schematic)
At the start: 89 parts, among them J2 0826-1X1T-HT-F, Q1 PSMN075-100MSE, Q2 PSMN075-100MSE, Q3 PSMN075-100MSE, Q4 PSMN075-100MSE, Q5 PSMN075-100MSE, Q6 PSMN075-100MSE, Q7 PSMN075-100MSE, Q8 PSMN075-100MSE, U1 MXL86211C-AQB-T, U2 TPS22917DBV, U3 TPS22917DBV, U4 SN74AXC4T774PWR, U5 LT4321xUF, X1 Q22FA23800194

Commit message: PoE Circuitry Updates.
Parts:
- removed C51: 47n, symbol Device:C_Small
- removed Q1, Q2, Q3, Q4, Q5, Q6, Q7, Q8: PSMN075-100MSE, klib_discrete:PSMN075-100MSE, symbol klib_discrete:PSMN075-100MSE
- removed R17: 0R, symbol Device:R
- removed U5: LT4321xUF, Package_DFN_QFN:QFN-16-1EP_4x4mm_P0.65mm_EP2.15x2.15mm, symbol Power_Management:LT4321xUF
- added C52, C53: 100n, Capacitor_SMD:C_0603_1608Metric, symbol Device:C_Small
- added R19, R20, R21, R22: 100R, Resistor_SMD:R_0603_1608Metric, symbol Device:R
- added R23: 0R, Resistor_SMD:R_0603_1608Metric, symbol Device:R
- added U6: SN74AXC4T774PWR, klib_logic:SN74AXC4T774PWR, symbol klib_logic:SN74AXC4T774PWR
Connections:
- net 1V8_FMC: now also C52.1, U6.16 (VCC_A)
- net 3V3_FMC: now also C53.1, U6.15 (VCC_B)
- net GND: now also C52.2, C53.2, R23.2, U6.10 (GND)
- net LED_0: now also R19.2
- net LED_1: now also R20.2
- net LED_2: now also R21.2
- net SHIFT_EN: now reaches R12.2, U4.9 (OE_N)
- net SHIFT_EN: now also R23.1, U6.9 (OE_N)
- new net: R20.1, U6.13 (B2)
- new net: R21.1, U6.12 (B3)
- new net: R22.1, U6.11 (B4)
- new net: R19.1, U6.14 (B1)
- new net L0_DIR: U6.1 (DIR1)
- new net L1_DIR: U6.2 (DIR2)
- new net L2_DIR: U6.7 (DIR3)
- new net LED_0_FMC: U6.3 (A1)
- new net LED_1_FMC: U6.4 (A2)
- new net LED_2_FMC: U6.5 (A3)
Other:
- added sheet POE_SUPPLY_12V_3A (POE_12V_3A.kicad_sch)
- moved on the sheet: C2, C3, C34, C35, C36, C37, C38, C39, C4, C40, C41, C42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

Commit message: Schematic Progress.
Connections:
- net GND: now also U6.8 (DIR4)
- net T2P_FLAG: now reaches U6.6 (A4)
- net T2P_FLAG: now also R22.2
Other:
- sheet POE_SUPPLY_12V_3A ports: added T2P_FLAG_ISO, T2P_FLAG_REF, V_AUX, V_OUT_12V; removed none
