File: 2G5_FMC_Test_Board_V1/POE_12V_3A.kicad_sch (KiCad schematic)
At the start: 38 parts, among them Q1 PSMN075-100MSE, Q10 PNP, Q2 PSMN075-100MSE, Q3 PSMN075-100MSE, Q4 PSMN075-100MSE, Q5 PSMN075-100MSE, Q6 PSMN075-100MSE, Q7 PSMN075-100MSE, Q8 PSMN075-100MSE, Q9 PSMN075-100MSE, U5 LT4321xUF, U7 LT4295xUFD

Commit message: Schematic Progress.
Parts:
- added C62, C65: 1u, symbol Device:C_Small
- added C63: 4n7, symbol Device:C_Small
- added C64, C75: 2n2, symbol Device:C_Small
- added C66: 100p, symbol Device:C_Small
- added C67: 22p, symbol Device:C_Small
- added C68: 220p, symbol Device:C_Small
- added C69, C70: 10u, symbol Device:C_Small
- added C71, C72: 47u, Package_DFN_QFN:WDFN-10-1EP_3x3mm_P0.5mm_EP1.8x2.5mm, symbol Device:C_Polarized_Small
- added C73: 3n3, symbol Device:C_Small
- added C74: 330p, symbol Device:C_Small
- added D5: BAT46WJ, Sensor_Humidity:Sensirion_DFN-4_1.5x1.5mm_P0.8mm_SHT4x_NoCentralPad, symbol Device:D_Schottky
- added D6: LED, LED_SMD:LED_Cree-XHP50_3V_HighDensity, symbol Device:LED
- added D8: PMEG1020EH, Diode_SMD:D_SOD-123F, symbol Diode:PMEG1020EH
- added JP1: SolderJumper_2_Open, Jumper:SolderJumper-2_P1.3mm_Open_Pad1.0x1.5mm, symbol Jumper:SolderJumper_2_Open
- added L10: 6mH, Inductor_THT:Choke_Schaffner_RN102-04-14.0x14.0mm, symbol Device:L_Coupled
- added L9: 220n, Relay_THT:Relay_DPDT_Finder_30.22, symbol Device:L
- added Q11: MMBT3904, Package_TO_SOT_SMD:SOT-23, symbol Transistor_BJT:MMBT3904
- added Q12: MMBT3906, Package_TO_SOT_SMD:SOT-23, symbol Transistor_BJT:MMBT3906
- added Q13, Q14: CSD18532NQ5B, Package_TO_SOT_SMD:TDSON-8-1, symbol Transistor_FET:CSD18532NQ5B
- added R33: 100R, Resistor_SMD:R_0603_1608Metric, symbol Device:R
- added R34, R49: 10k, symbol Device:R
- added R35: 15R, Resistor_SMD:R_0603_1608Metric, symbol Device:R
- added R36, R37: 39, symbol Device:R
- added R38: 20m, symbol Device:R
- added R39, R40, R41: 0R, Resistor_SMD:R_0603_1608Metric, symbol Device:R
- added R42, R43: 75R, symbol Device:R
- added R44: 5k62, symbol Device:R
- added R45: 2k, symbol Device:R
- added R46: 4k7, symbol Device:R
- added R47: 30k, symbol Device:R
- added R48: 4k7, Resistor_SMD:R_0603_1608Metric, symbol Device:R
- added T1: PE-68386NL, Transformer_SMD:Pulse_PA2001NL, symbol Transformer:PE-68386NL
- added U8: TLP291, Package_SO:SOIC-4_4.55x2.6mm_P1.27mm, symbol Isolator:TLP291
- added X2: 750316116, klib_discrete:750316116, symbol klib_discrete:750316116
- C54: V 100V -> 25V
- C55: value 100n -> 100p
- C56: value ? -> 47n
- C57: value ? -> 10n
- C59, C60: value ? -> 2u2
- C61: value ? -> 10u; V 100V -> 10V
- D1, D4: value D_TVS -> PTVS58VS1UR
- D3: value D -> BAV19WS
- L7: value L -> 4u7
- L8: value L -> 100u
- Q10: value PNP -> FMMT723
- R18: value ? -> 47R5
- R24: value ? -> 150R
- R25: value ? -> 10k
- R26: value ? -> 107k
- R27: value ? -> 52k3
- R28: value ? -> 174k
- R29: value ? -> 8R2
- R30: value ? -> 3k3
- R31: value ? -> 5k23
- R32: value ? -> 20R
Connections:
- net GND is gone; now on net VPORT_N: C54.1, C55.1, C56.1, C57.1, C58.2, C59.1, C60.1, C61.1, D1.1 (A1), D3.2 (A), D4.1 (A1), R18.2, R24.2, R25.2, R26.2, R27.2, R31.2, U7.1 (GND), U7.19 (GND), U7.29 (GND)
- net VPORT_N: now also C63.1, C74.1, D8.2 (A), L10.4, R38.2, R40.2, R45.2, R47.2, T1.3, U8.2, X2.5; no longer Q2.1, Q2.2, Q2.3, Q4.1, Q4.2, Q4.3, Q6.1, Q6.2, Q6.3, Q8.1, Q8.2, Q8.3
- net VPORT_P: now also D1.2 (A2), Q9.MB, R29.1, L10.2; no longer Q1.MB, Q3.MB, Q5.MB, Q7.MB
- net V_PRIMARY: now also C59.2, C60.2, D4.2 (A2), L7.2, U7.24 (VIN), C75.1, R42.1, R43.1, X2.1, X2.2
- net V_AUX: now reaches D2.2 (A), R28.1
- net at R25.1: now also JP1.1 (A); no longer U7.15 (RLDCMP)
- net at U7.13 (ITHB): now also C73.2, C74.2
- net at U7.14 (FB31): now also R44.2, R45.1
- net at U7.16 (ISEN-): now also C67.1, R40.1
- net at U7.17 (ISEN+): now also C67.2, R39.1
- net at U7.18 (SG): now also R33.1
- net at U7.20 (PG): now also D8.1 (K), R41.1
- net T2P_FLAG: now reaches U7.5 (T2P)
- net T2P_FLAG: now also R48.1
- new net: C68.2, R42.2, R43.2
- new net: R48.2, U8.1
- new net: C66.2, C75.2, Q13.5 (D), X2.11, X2.12
- new net: C68.1, Q14.5 (D), X2.3, X2.4
- new net: C69.2, C70.2, L9.1, X2.7, X2.8
- new net: JP1.2 (B), U7.15 (RLDCMP)
- new net: Q11.1 (B), Q12.1 (B), R35.2
- new net: Q11.2 (E), Q12.2 (E), Q13.4 (G)
- new net: Q14.1 (S), Q14.2 (S), Q14.3 (S), R38.1, R39.2
- new net: D6.2 (A), R46.2
- new net: C64.2, D5.1 (K), R34.1, R35.1
- new net: C62.1, R33.2
- new net: C62.2, T1.1
- new net: C66.1, R36.1, R37.1
- new net: C64.1, T1.6
- new net: L10.3, Q2.1, Q2.2, Q2.3, Q4.1, Q4.2, Q4.3, Q6.1, Q6.2, Q6.3, Q8.1, Q8.2, Q8.3
- new net: L10.1, Q1.MB, Q3.MB, Q5.MB, Q7.MB
- new net: Q14.4 (G), R41.2
- new net: C73.1, R47.1
- new net FB: R44.1, X2.6
- new net GND1: C63.2, C65.1, C69.1, C70.1, C71.2, C72.2, D5.2 (A), D6.1 (K), Q12.3 (C), Q13.1 (S), Q13.2 (S), Q13.3 (S), R34.2, R36.2, R37.2, T1.4, U8.3
- new net T2P_FLAG_ISO: R49.2, U8.4
- new net T2P_FLAG_REF: R49.1
- new net V_OUT_12V: C65.2, C71.1, C72.1, L9.2, Q11.3 (C), R46.1
Other:
- moved on the sheet: C51, C54, C55, C56, C57, C58, C59, C60, C61, D1, D2, D3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
